File: hardware/kicad/Hyperloop-TB-Circuit/Hyperloop-TB-Circuit.kicad_sch (KiCad schematic)
At the start: 0 parts

Commit message: Finishing kicad drawing
Parts:
- added J1: Conn_01x02, symbol Connector_Generic:Conn_01x02
Changed lines of the file:
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@@
 	(generator_version "9.0")
 	(paper "A4")
+	(symbol
+		(lib_id "Connector_Generic:Conn_01x02")
+		(at 63.5 93.98 0)
+		(unit 1)
+		(exclude_from_sim no)
+		(in_bom yes)
+		(on_board yes)
+		(dnp no)
+		(fields_autoplaced yes)
+		(property "Reference" "J1"
+			(at 66.04 93.9799 0)
+			(effects
+				(font
+					(size 1.27 1.27)
+				)
+				(justify left)
+			)
+		)
+		(property "Value" "Conn_01x02"
+			(at 66.04 96.5199 0)
+			(effects
+				(font
+					(size 1.27 1.27)
+				)
+				(justify left)
+			)
+		)
+		(property "Footprint" ""
+			(at 63.5 93.98 0)
+			(effects
+				(font
+					(size 1.27 1.27)
+				)
+				(hide yes)
+			)
+		)
+		(property "Datasheet" "~"
+			(at 63.5 93.98 0)
+			(effects
+				(font
+					(size 1.27 1.27)
+				)
+				(hide yes)
+			)
+		)
+		(property "Description" "Generic connector, single row, 01x02, script generated (kicad-library-utils/schlib/autogen/connector/)"
+			(at 63.5 93.98 0)
+			(effects
+				(font
+					(size 1.27 1.27)
+				)
+				(hide yes)
+			)
+		)
+		(pin "1"
+		)
+		(pin "2"
+		)
+		(instances
+			(project ""
+				(path "/892d4e79-3353-4dfb-9ceb-97f2ebb2dd36"
+					(reference "J1")
+					(unit 1)
+				)
+			)
+		)
+	)
 	(sheet_instances
 		(path "/"

Commit message: Halfway
Parts:
- added C1: 100NF, symbol Device:C
- added C2, C3: 220NF, symbol Device:C
- added D1: 1N4001, Diode_THT:D_DO-41_SOD81_P10.16mm_Horizontal, symbol Diode:1N4001
- added J2: Conn_01x02, symbol Connector_Generic:Conn_01x02
- added PS1: SDM30-24S5, SDM30-24S5:CONV_SDM30-24S5, symbol New_Library:SDM30-24S5
- added Q1: IRLZ44N, symbol New_Library:IRLZ44N
Connections:
- net +24V: now reaches J1.1 (Pin_1)
- net +24V: now also C1.1, PS1.1 (+VIN)
- net GND: now reaches J1.2 (Pin_2)
- net GND: now also C1.2, C2.2, C3.2, PS1.2 (-VIN), PS1.7 (-VOUT), Q1.3 (SOURCE)
- new net: D1.2 (A), J2.2 (Pin_2), Q1.2 (DRAIN)
- new net +5V: C2.1, C3.1, D1.1 (K), J2.1 (Pin_1), PS1.6 (+VOUT)
- new net MOTOR_GATE: Q1.1 (GATE)
Other:
- moved on the sheet: J1

Commit message: Pushing file for Jacob
Parts:
- added R1: 20K Ohms, symbol Device:R
- added R2: 10K Ohms, symbol Device:R
- added R3: 100 ohms, symbol Device:R
- added R4: 100k ohms, symbol Device:R
- added Teensy: Conn_01x06_Pin, symbol Connector:Conn_01x06_Pin
Connections:
- net +5V: now also Teensy.1 (Pin_1)
- net GND: now also R1.2, R4.1, Teensy.2 (Pin_2), Teensy.3 (Pin_3)
- new net: R3.1, R4.2
- new net: R3.2, Teensy.4 (Pin_4)
- new net ECHO: R1.1, R2.2, Teensy.6 (Pin_6)
- new net ECHO_RAW: R2.1
- new net TRIG: Teensy.5 (Pin_5)

Commit message: saved
Parts:
- renumbered Teensy to Teensy1
Changed lines of the file:
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@@
 		(on_board yes)
 		(dnp no)
-		(property "Reference" "Teensy"
+		(property "Reference" "Teensy1"
 			(at 229.235 116.84 0)
 			(effects
@@
 			(project ""
 				(path "/892d4e79-3353-4dfb-9ceb-97f2ebb2dd36"
-					(reference "Teensy")
+					(reference "Teensy1")
 					(unit 1)
 				)

Commit message: Connected Resistor Footprints to schematic
Parts:
- Q1: footprint (none) -> TB-Footprint_Lib:IFX-PG-TO220-3-904-1
- R1, R2, R3, R4: footprint (none) -> Resistor_THT:R_Axial_DIN0204_L3.6mm_D1.6mm_P7.62mm_Horizontal
Changed lines of the file:
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@@
 			)
 		)
-		(property "Footprint" ""
+		(property "Footprint" "Resistor_THT:R_Axial_DIN0204_L3.6mm_D1.6mm_P7.62mm_Horizontal"
 			(at 215.9 131.318 90)
 			(effects
@@
 			)
 		)
-		(property "Footprint" ""
+		(property "Footprint" "Resistor_THT:R_Axial_DIN0204_L3.6mm_D1.6mm_P7.62mm_Horizontal"
 			(at 208.788 137.16 90)
 			(effects
@@
 			)
 		)
-		(property "Footprint" ""
+		(property "Footprint" "Resistor_THT:R_Axial_DIN0204_L3.6mm_D1.6mm_P7.62mm_Horizontal"
 			(at 46.99 128.778 90)
 			(effects
@@
 			)
 		)
-		(property "Footprint" ""
+		(property "Footprint" "TB-Footprint_Lib:IFX-PG-TO220-3-904-1"
 			(at 168.91 49.53 0)
 			(effects
@@
 			)
 		)
-		(property "Footprint" ""
+		(property "Footprint" "Resistor_THT:R_Axial_DIN0204_L3.6mm_D1.6mm_P7.62mm_Horizontal"
 			(at 32.512 134.62 90)
 			(effects

Commit message: Connected all the parts to a footprint schematic
Parts:
- C1, C2, C3: footprint (none) -> Capacitor_THT:C_Disc_D6.0mm_W2.5mm_P5.00mm
- J1, J2: footprint (none) -> Connector_PinHeader_1.00mm:PinHeader_1x02_P1.00mm_Vertical
- PS1: footprint SDM30-24S5:CONV_SDM30-24S5 -> TB-Footprint_Lib:CONV_SDM30-24S5
- Teensy1: footprint (none) -> Connector_PinHeader_1.00mm:PinHeader_1x06_P1.00mm_Vertical
Changed lines of the file:
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@@
 			)
 		)
-		(property "Footprint" ""
+		(property "Footprint" "Capacitor_THT:C_Disc_D6.0mm_W2.5mm_P5.00mm"
 			(at 125.4252 92.71 0)
 			(effects
@@
 			)
 		)
-		(property "Footprint" ""
+		(property "Footprint" "Connector_PinHeader_1.00mm:PinHeader_1x06_P1.00mm_Vertical"
 			(at 229.87 127 0)
 			(effects
@@
 			)
 		)
-		(property "Footprint" ""
+		(property "Footprint" "Connector_PinHeader_1.00mm:PinHeader_1x02_P1.00mm_Vertical"
 			(at 26.67 87.63 0)
 			(effects
@@
 			)
 		)
-		(property "Footprint" ""
+		(property "Footprint" "Capacitor_THT:C_Disc_D6.0mm_W2.5mm_P5.00mm"
 			(at 39.0652 92.71 0)
 			(effects
@@
 			)
 		)
-		(property "Footprint" ""
+		(property "Footprint" "Capacitor_THT:C_Disc_D6.0mm_W2.5mm_P5.00mm"
 			(at 112.7252 92.71 0)
 			(effects
@@
 			)
 		)
-		(property "Footprint" "SDM30-24S5:CONV_SDM30-24S5"
+		(property "Footprint" "TB-Footprint_Lib:CONV_SDM30-24S5"
 			(at 74.93 88.9 0)
 			(effects
@@
 			)
 		)
-		(property "Footprint" ""
+		(property "Footprint" "Connector_PinHeader_1.00mm:PinHeader_1x02_P1.00mm_Vertical"
 			(at 182.88 60.96 0)
 			(effects
