File: hardware/kicad/Hyperloop-TB-Circuit/Hyperloop-TB-Circuit.kicad_pcb (KiCad board)
At the start: 2 copper layers, 1 part

Commit message: updated schematic and pcb
Parts:
- removed D1: 1N4001, Diode_THT:D_DO-41_SOD81_P10.16mm_Horizontal
- added C1: 100NF, Capacitor_THT:C_Disc_D3.0mm_W1.6mm_P2.50mm, F.Cu at (148.6, 91.0)
- added C2: 220NF, Capacitor_THT:C_Disc_D3.0mm_W1.6mm_P2.50mm, F.Cu at (148.6, 94.2)
- added C3: 220NF, Capacitor_THT:C_Disc_D3.0mm_W1.6mm_P2.50mm, F.Cu at (148.6, 97.3)
- added J1: Conn_01x02, Connector_PinHeader_1.00mm:PinHeader_1x02_P1.00mm_Vertical, F.Cu at (148.7, 108.5)
- added J2: Conn_01x02, Connector_PinHeader_1.00mm:PinHeader_1x02_P1.00mm_Vertical, F.Cu at (152.0, 108.5)
- added J3: Conn_01x04_Pin, Connector_Samtec_HPM_THT:Samtec_HPM-04-01-x-S_Straight_1x04_Pitch5.08mm, F.Cu at (151.2, 70.7)
- added PS1: SDM30-24S5, TB-Footprint_Lib:CONV_SDM30-24S5, F.Cu at (120.3, 93.3)
- added Q1: IRLZ44N, TB-Footprint_Lib:IFX-PG-TO220-3-904-1, F.Cu at (100.6, 123.0)
- added R1: 20K Ohms, Resistor_THT:R_Axial_DIN0204_L3.6mm_D1.6mm_P7.62mm_Horizontal, F.Cu at (107.8, 121.0)
- added R2: 10K Ohms, Resistor_THT:R_Axial_DIN0204_L3.6mm_D1.6mm_P7.62mm_Horizontal, F.Cu at (66.7, 120.0)
- added Teensy1: Conn_01x06_Pin, Connector_PinHeader_1.00mm:PinHeader_1x06_P1.00mm_Vertical, F.Cu at (148.7, 100.5)
Routing:
- net Net-(J2-Pin_2): track 0.00 -> 145.9 mm
- net Net-(J3-Pin_4): track 0.00 -> 139.7 mm, vias 0 -> 1
- net /TRIG: track 0.00 -> 115.6 mm, vias 0 -> 1
- net +5V: track 0.00 -> 95.9 mm
- net Net-(Q1-GATE): track 0.00 -> 94.5 mm, vias 0 -> 1
- net /ECHO: track 0.00 -> 81.4 mm
- net GND: track 0.00 -> 25.9 mm, vias 0 -> 1
- net +24V: track 0.00 -> 23.9 mm
- added copper zone on B.Cu, net GND

Commit message: new pcb
Parts:
- moved R2 115.6 mm to (182.3, 122.8)
- moved Q1 74.5 mm to (175.1, 121.6)
- moved R1 74.5 mm to (182.3, 119.7)
- moved C1 23.6 mm to (171.6, 96.5)
- moved C2 23.6 mm to (171.6, 99.7)
- moved C3 23.6 mm to (171.6, 102.8)
- moved J1 23.6 mm to (171.7, 114.0)
- moved J2 23.6 mm to (175.0, 114.0)
- moved J3 23.6 mm to (174.2, 76.2)
- moved PS1 23.6 mm to (143.3, 98.8)
- moved Teensy1 23.6 mm to (171.7, 106.0)
Routing:
- net Net-(J3-Pin_4): track 139.7 -> 34.8 mm, vias 1 -> 0
- net Net-(J2-Pin_2): track 145.9 -> 50.9 mm
- net /TRIG: track 115.6 -> 25.2 mm, vias 1 -> 0
- net GND: track 25.9 -> 115.6 mm, vias 1 -> 0
- net /ECHO: track 81.4 -> 29.8 mm
- net Net-(Q1-GATE): track 94.5 -> 51.7 mm, vias 1 -> 0
- net +5V: track 95.9 -> 128.1 mm
- removed copper zone on B.Cu, net GND
Other:
- board outline added: 77 x 56 mm
